File: PCB/KosmicSuperspreader.sch (KiCad schematic (older format))
At the start: 28 parts, among them J1 CV INPUT, J2 SPREAD INPUT, J3 OUT -, J4 OUT +, J5 BUFFER, J6 SYNTH POWER, U1 TL072, U2 TL074

Commit message: sch pdf to docs
Other:
- note removed: "NOT TESTED!"
Changed lines of the file:
@@
 Text Notes 3650 1850 0    50   ~ 0
 spreader circuit
-Text Notes 950  1350 0    394  ~ 79
-NOT TESTED!
 $Comp
 L power:GND #PWR0106

Commit message: gerbs
Connections:
- net +12V: now also RV2.3; no longer RV2.1
- net GND: now also RV1.1, RV2.1; no longer RV1.3, RV2.3
- net SPREAD: now also RV1.3; no longer RV1.1
Changed lines of the file:
@@
 F 3 "~" H 3300 3700 50  0001 C CNN
 	1    3300 3700
-	1    0    0    -1
+	1    0    0    1
 $EndComp
 Text GLabel 9250 3400 2    50   Input ~ 0
@@
 F 3 "~" H 3300 2950 50  0001 C CNN
 	1    3300 2950
-	1    0    0    -1
+	1    0    0    1
 $EndComp
 $Comp
